File: gl852.kicad_pcb (KiCad board)
At the start: 2 copper layers, 100 x 100 mm, 98 parts, among them J1 USB_B, J10 USB_A, J11 USB_A, J12 USB_A, J2 12V, J3 VBUS, J4 3V3, J5 VBUS_34, J6 VBUS_12, J9 USB_A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

Commit message: Modified power section
Parts:
- removed C29, C31: 100n, Capacitor_SMD:C_0603_1608Metric_Pad1.08x0.95mm_HandSolder
- removed Q2: BC817, Package_TO_SOT_SMD:SOT-23
- removed R26: 100R, Resistor_SMD:R_0603_1608Metric_Pad0.98x0.95mm_HandSolder
- added D7: Self Power, LED_SMD:LED_0805_2012Metric_Pad1.15x1.40mm_HandSolder, F.Cu at (35.0, 26.9)
- added D8: MBRA340T3G, Diode_SMD:D_SMC_Handsoldering, F.Cu at (24.1, 45.9)
- added D9: Ext Power, LED_SMD:LED_0805_2012Metric_Pad1.15x1.40mm_HandSolder, F.Cu at (37.7, 26.9)
- added J7: 5VExt, Connector_PinHeader_2.54mm:PinHeader_1x02_P2.54mm_Vertical, F.Cu at (4.45, 86.5)
- added R27: 1k, Resistor_SMD:R_0603_1608Metric_Pad0.98x0.95mm_HandSolder, F.Cu at (32.9, 27.0)
- added U12: 74LVC1G06, Package_TO_SOT_SMD:SOT-23-5_HandSoldering, F.Cu at (29.6, 35.3)
- J3: footprint Connector_PinHeader_2.54mm:PinHeader_2x02_P2.54mm_Vertical -> Connector_PinHeader_2.54mm:PinHeader_1x02_P2.54mm_Vertical
- J4: value 3V3 -> 3.3V; footprint Connector_PinHeader_2.54mm:PinHeader_2x02_P2.54mm_Vertical -> Connector_PinHeader_2.54mm:PinHeader_1x02_P2.54mm_Vertical
- Q3: value AO3401A -> IRLML6402
- R24: value 10k -> 100k
- U6: value LM358 -> 74LVC1G06; footprint Package_SO:SOIC-8_3.9x4.9mm_P1.27mm -> Package_TO_SOT_SMD:SOT-23-5_HandSoldering
- Y1: value Crystal -> 12 MHz
- moved R25 39.7 mm to (39.8, 26.9), turned to 90 degrees
- moved C1 19.0 mm to (54.0, 69.2), turned to -90 degrees
- moved C4 18.4 mm to (58.9, 69.2), turned to -90 degrees
- moved R23 15.8 mm to (29.8, 57.9)
- moved U6 14.9 mm to (24.1, 35.3), turned to 90 degrees
- moved Y1 12.1 mm to (54.0, 64.0), turned to 0 degrees
- moved J3 6.98 mm to (32.9, 4.88), turned to 0 degrees
- moved R24 4.60 mm to (29.6, 39.6), turned to -90 degrees
- moved Q3 1.70 mm to (26.7, 57.9)
- moved J4 1.64 mm to (25.6, 4.88), turned to 0 degrees
Connections:
- L9 pad 2: /5V_EXT -> /GATE_CMD
- L9 pad 3: /5V_EXT -> /GATE_CMD
- R23 pad 1: /+12V_IN -> GND
- R23 pad 2: /CMP -> /GATE_CMD
- R24 pad 1: /CMP -> Net-(D7-Pad1)
- R24 pad 2: GND -> +3V3
- R25 pad 1: /GATE_CMD -> Net-(D9-Pad2)
- R25 pad 2: Net-(Q2-Pad1) -> /5V_EXT
- U6 pad 1: Net-(U6-Pad1) -> (no net)
- U6 pad 2: /5V_EXT -> /GATE_CMD
- U6 pad 3: /CMP -> GND
- U6 pad 4: GND -> Net-(D7-Pad1)
- U6 pad 5: Net-(U6-Pad1) -> +3V3
Routing:
- net /+12V_IN: track 109.9 -> 52.8 mm, vias 2 -> 0
- net /GATE_CMD: track 11.9 -> 61.3 mm
- net /5V_EXT: track 267.8 -> 305.2 mm, vias 4 -> 5
- net /PSELF: track 80.0 -> 48.8 mm
- net Net-(D7-Pad1): track 0.00 -> 23.6 mm
- net /X2: track 26.2 -> 17.9 mm, vias 1 -> 0
- net Net-(U6-Pad1): track 7.46 -> 0.00 mm
- net /CMP: track 7.15 -> 0.00 mm
- net /D1_N: track 69.9 -> 63.0 mm
- net /D1_P: track 68.3 -> 63.0 mm
- net /X1: track 26.4 -> 21.2 mm, vias 1 -> 0
- net GND: track 132.9 -> 127.8 mm, vias 34 -> 33
- net /VBUS: track 184.4 -> 188.9 mm
- net /D0_N: track 44.2 -> 48.2 mm
- net Net-(Q2-Pad1): track 3.93 -> 0.00 mm
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Other:
- board text added: "5V Ext"
- board text added: "GND"
- board text added: "Port 1"
- board text added: "Port 2"
- board text added: "Port 3"
- board text added: "Port 4"
- board text added: "Reset"
- board text added: "SUSPEND"
- board text added: "Self"
- board text added: "V+"
- board text added: "V-"
