File: gl852.kicad_sch (KiCad schematic)
At the start: 98 parts, among them J1 USB_B, J10 USB_A, J11 USB_A, J12 USB_A, J2 12V, J3 VBUS, J4 3V3, J5 VBUS_34, J6 VBUS_12, J9 USB_A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

Commit message: Modified power section
Parts:
- removed C29, C31: 100n, Capacitor_SMD:C_0603_1608Metric_Pad1.08x0.95mm_HandSolder, symbol areal_hlk_7621-rescue:C-Device
- removed J3: VBUS, Connector_PinHeader_2.54mm:PinHeader_2x02_P2.54mm_Vertical, symbol Connector_Generic:Conn_02x02_Odd_Even
- removed J4: 3V3, Connector_PinHeader_2.54mm:PinHeader_2x02_P2.54mm_Vertical, symbol Connector_Generic:Conn_02x02_Odd_Even
- removed Q2: BC817, Package_TO_SOT_SMD:SOT-23, symbol Transistor_BJT:BC817
- removed R23, R24: 10k, Resistor_SMD:R_0603_1608Metric_Pad0.98x0.95mm_HandSolder, symbol areal_hlk_7621-rescue:R-Device
- removed R26: 100R, Resistor_SMD:R_0603_1608Metric_Pad0.98x0.95mm_HandSolder, symbol areal_hlk_7621-rescue:R-Device
- removed U6: LM358, Package_SO:SOIC-8_3.9x4.9mm_P1.27mm, symbol Amplifier_Operational:LM358
- added D7: Self Power, LED_SMD:LED_0805_2012Metric_Pad1.15x1.40mm_HandSolder, symbol Device:LED
- added D8: MBRA340T3G, Diode_SMD:D_SMC_Handsoldering, symbol areal_hlk_7621-rescue:MBR340-Diode
- added D9: Ext Power, LED_SMD:LED_0805_2012Metric_Pad1.15x1.40mm_HandSolder, symbol Device:LED
- added J3: VBUS, Connector_PinHeader_2.54mm:PinHeader_1x02_P2.54mm_Vertical, symbol Connector:Conn_01x02_Male
- added J4: 3.3V, Connector_PinHeader_2.54mm:PinHeader_1x02_P2.54mm_Vertical, symbol Connector:Conn_01x02_Male
- added J7: 5VExt, Connector_PinHeader_2.54mm:PinHeader_1x02_P2.54mm_Vertical, symbol Connector:Conn_01x02_Male
- added R23: 10k, Resistor_SMD:R_0603_1608Metric_Pad0.98x0.95mm_HandSolder, symbol Device:R
- added R24: 100k, Resistor_SMD:R_0603_1608Metric_Pad0.98x0.95mm_HandSolder, symbol Device:R
- added R27: 1k, Resistor_SMD:R_0603_1608Metric_Pad0.98x0.95mm_HandSolder, symbol areal_hlk_7621-rescue:R-Device
- added U12, U6: 74LVC1G06, Package_TO_SOT_SMD:SOT-23-5_HandSoldering, symbol 74xGxx:74LVC1G06
- Q3: value AO3401A -> IRLML6402
- Y1: value Crystal -> 12 MHz
Connections:
- net +3V3: now also J4.1 (Pin_1), R24.2, R27.2, U12.5 (VCC), U6.5 (VCC)
- net 5V_EXT: now also R25.2, D8.1 (K), J7.1 (Pin_1); no longer L9.2, L9.3
- net GATE_CMD: now also L9.2, L9.3, D8.2 (A), R23.2, U6.2; no longer R25.1
- net GND: now also D9.1 (K), J3.2 (Pin_2), J4.2 (Pin_2), J7.2 (Pin_2), R23.1, U12.3 (GND), U6.3 (GND)
- net PSELF: now also U12.4
- net VBUS: now also J3.1 (Pin_1)
- new net: D7.1 (K), R24.1, U12.2, U6.4
- new net: D7.2 (A), R27.1
- new net: D9.2 (A), R25.1
Other:
- moved on the sheet: C24, C25, C26, C27, C28, D5, D6, J2, L1, L8, L9, Q1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
